File: universal12Vsupply/universal12Vsupply.kicad_sch (KiCad schematic)
At the start: 66 parts, among them J1 Screw_Terminal_01x04, J2 Screw_Terminal_01x02, U1 LM5175PWP

Commit message: started PCB layout
Parts:
- added C7, C8, C9: 15u, Capacitor_SMD:C_1206_3216Metric_Pad1.33x1.80mm_HandSolder, symbol Device:C
- renumbered Rsense to Rsense1
Connections:
- net GND: now also C7.2, C8.2, C9.2
- net Vin: now also C7.1, C8.1, C9.1
Other:
- moved on the sheet: C2, Cin1, D3, H1, H2, H3, H4, J1, J2, R1, R2, R3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

Commit message: 'finalised' layout without DRC errors
Parts:
- L1: footprint Inductor_SMD:L_Coilcraft_XAL1010-XXX -> FootprintLibrary:L_Coilcraft_XAL1010-XXX_handsolder
Changed lines of the file:
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@@
       (effects (font (size 1.27 1.27)))
     )
-    (property "Footprint" "Inductor_SMD:L_Coilcraft_XAL1010-XXX" (at 279.4 50.8 0)
+    (property "Footprint" "FootprintLibrary:L_Coilcraft_XAL1010-XXX_handsolder" (at 279.4 50.8 0)
       (effects (font (size 1.27 1.27)) hide)
     )
