File: universal12Vsupply/universal12Vsupply.kicad_sch (KiCad schematic)
At the start: 62 parts, among them J1 Screw_Terminal_01x04, J2 Screw_Terminal_01x02, SW1 TestPoint, U1 LM5175PWP

Commit message: added test points properly, DRC and ERC is fine
Parts:
- removed SW1, TP14, source2_4: TestPoint, TestPoint:TestPoint_THTPad_2.5x2.5mm_Drill1.2mm, symbol Connector:TestPoint
- added TP1: LDRV2, TestPoint:TestPoint_THTPad_2.5x2.5mm_Drill1.2mm, symbol Connector:TestPoint
- added TP10: Vin, TestPoint:TestPoint_THTPad_2.5x2.5mm_Drill1.2mm, symbol Connector:TestPoint
- added TP6: LDRV1, TestPoint:TestPoint_THTPad_2.5x2.5mm_Drill1.2mm, symbol Connector:TestPoint
- TP11: renamed from TP10; value TestPoint -> gnd
- TP12: renamed from TP11; value TestPoint -> gnd
- TP13: renamed from TP12; value TestPoint -> gnd
- TP14: renamed from TP13; value TestPoint -> gnd
- TP15: value TestPoint -> source2_4
- TP2: value TestPoint -> ICVin
- TP3: value TestPoint -> Vcc
- TP4: value TestPoint -> HDRV1
- TP5: value TestPoint -> SW1
- TP7: value TestPoint -> HDRV2
- TP8: value TestPoint -> SW2
- TP9: value TestPoint -> Vout
Connections:
- net HDRV1: now also TP4.1; no longer TP5.1
- net HDRV2: now also TP7.1; no longer TP8.1
- net ICVin: now also TP2.1; no longer TP3.1
- net LDRV1: now also TP6.1; no longer TP7.1
- net LDRV2: now also TP1.1; no longer TP2.1
- net SW1: now also TP5.1
- net SW2: now also TP8.1; no longer TP9.1
- net Vcc: now also TP3.1; no longer TP4.1
- net Vin: now also TP10.1; no longer TP15.1
- net Vout: now also TP9.1
- net source2_4: now also TP15.1

Commit message: finished PCB
Parts:
- added Cbias1: 100n, Capacitor_SMD:C_0805_2012Metric_Pad1.18x1.45mm_HandSolder, symbol Device:C
- H1, H2, H3, H4, TP1, TP10, TP11, TP12, TP13, TP14, TP15, TP2, TP3, TP4, TP5, TP6, TP7, TP8, TP9: now left out of the parts list
- renumbered Cbias1 to Cvcc1
Connections:
- net GND: now also Cvcc1.2, Cbias1.2
- net Vout: now also U1.24 (BIAS), Cbias1.1
- removed net BIAS: Cvcc1.2, U1.24 (BIAS)
Other:
- moved on the sheet: C2, Cboot1, Cvcc1, D3, Dboot1, R1, R2, R3
