File: universal12Vsupply/universal12Vsupply.kicad_sch (KiCad schematic)
At the start: 64 parts, among them J1 Screw_Terminal_01x04, J2 Screw_Terminal_01x02, U1 LM5175PWP

Commit message: added design report i think
Parts:
- C3, C4, C6, C7, C8, C9: symbol Device:C -> Device:C_Polarized
Changed lines of the file:
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@@
     )
   )
-  (symbol (lib_id "Device:C") (at 327.66 40.64 0) (unit 1)
+  (symbol (lib_id "Device:C_Polarized") (at 327.66 40.64 0) (unit 1)
     (in_bom yes) (on_board yes) (dnp no)
     (property "Reference" "C4" (at 328.93 38.1 0)
@@
     )
   )
-  (symbol (lib_id "Device:C") (at 335.28 40.64 0) (unit 1)
+  (symbol (lib_id "Device:C_Polarized") (at 335.28 40.64 0) (unit 1)
     (in_bom yes) (on_board yes) (dnp no)
     (property "Reference" "C6" (at 336.55 38.1 0)
@@
     )
   )
-  (symbol (lib_id "Device:C") (at 320.675 40.64 0) (unit 1)
+  (symbol (lib_id "Device:C_Polarized") (at 320.675 40.64 0) (unit 1)
     (in_bom yes) (on_board yes) (dnp no)
     (property "Reference" "C3" (at 321.945 38.1 0)
@@
     )
   )
-  (symbol (lib_id "Device:C") (at 57.785 128.905 0) (unit 1)
+  (symbol (lib_id "Device:C_Polarized") (at 57.785 128.905 0) (unit 1)
     (in_bom yes) (on_board yes) (dnp no)
     (property "Reference" "C7" (at 59.055 126.365 0)
@@
     )
   )
-  (symbol (lib_id "Device:C") (at 72.39 128.905 0) (unit 1)
+  (symbol (lib_id "Device:C_Polarized") (at 72.39 128.905 0) (unit 1)
     (in_bom yes) (on_board yes) (dnp no)
     (property "Reference" "C9" (at 73.66 126.365 0)
@@
     )
   )
-  (symbol (lib_id "Device:C") (at 64.77 128.905 0) (unit 1)
+  (symbol (lib_id "Device:C_Polarized") (at 64.77 128.905 0) (unit 1)
     (in_bom yes) (on_board yes) (dnp no)
     (property "Reference" "C8" (at 66.04 126.365 0)
